Commit message: control.launch.py appears to be failing because loader not found for the custom controllers. troubleshooting that now

File: ridgeback_description/urdf/accessories.urdf.xacro (robot description, xacro)
@@ -9,5 +9,5 @@
     ridgeback_base/launch/base.launch
   -->
-  <xacro:include filename="$(find ridgeback_description)/urdf/accessories/sick_lms1xx_mount.urdf.xacro" />
+<!--  <xacro:include filename="$(find ridgeback_description)/urdf/accessories/sick_lms1xx_mount.urdf.xacro" />-->
   <xacro:include filename="$(find ridgeback_description)/urdf/accessories/sick_s300_mount.urdf.xacro" />
   <xacro:include filename="$(find ridgeback_description)/urdf/accessories/hokuyo_ust-10lx_mount.urdf.xacro" />
@@ -25,15 +25,15 @@
   </xacro:if>
   <!-- If enabled, generate the front SICK LMS111 LASER payload. -->
-  <xacro:if value="$(optenv RIDGEBACK_FRONT_SICK_LASER 0)">
+<!--  <xacro:if value="$(optenv RIDGEBACK_FRONT_SICK_LASER 0)">
     <xacro:sick_lms1xx_mount prefix="front"
                              topic="front/scan"
                              location="1" />
-  </xacro:if>
+  </xacro:if>-->
   <!-- If enabled, generate the rear SICK LMS111 LASER payload. -->
-  <xacro:if value="$(optenv RIDGEBACK_REAR_SICK_LASER 0)">
+<!--  <xacro:if value="$(optenv RIDGEBACK_REAR_SICK_LASER 0)">
     <xacro:sick_lms1xx_mount prefix="rear"
                              topic="rear/scan"
                              location="-1" />
-  </xacro:if>
+  </xacro:if>-->
   <!-- If enabled, generate the front SICK S300 LASER payload.
        This uses the same mesh as the lms1xx since they are the footprint

File: ridgeback_description/urdf/ridgeback.urdf.xacro (robot description, xacro)
@@ -1,4 +1,5 @@
 <?xml version="1.0"?>
 <robot name="ridgeback" xmlns:xacro="http://ros.org/wiki/xacro">
+  <xacro:arg name="use_fake_hardware" default="true"/>
   <xacro:property name="PI" value="3.1415926535897931" />
   <xacro:property name="wheel_radius" value="0.0759" />
@@ -21,4 +22,13 @@
   <material name="yellow"><color rgba="0.8 0.8 0.0 1.0" /></material>
   <material name="black"><color rgba="0.15 0.15 0.15 1.0" /></material>
+  <!-- ros2 control include -->
+  <!-- xacro:include filename="$(find ridgeback_description)/urdf/ridgeback.ros2_control.xacro" /-->
+  <!-- ros2 control instance -->
+  <!-- xacro:ridgeback_ros2_control
+    name="ridgeback_ros2_control" prefix="${prefix}"
+    side="${side}"
+    use_fake_hardware="$(arg use_fake_hardware)"
+    initial_positions="${initial_positions}"
+    robot_ip="$(arg robot_ip)" /-->
   <xacro:macro name="wheel" params="prefix side *joint_pose">
     <link name="${prefix}_${side}_wheel_link">
@@ -264,4 +274,38 @@
     <origin xyz="0 0 ${deck_height}" rpy="0 0 0"/>
   </joint>
+  <ros2_control name="ridgeback_hardware" type="system">
+    <hardware>
+      <xacro:if value="$(arg use_fake_hardware)">
+        <plugin>fake_components/GenericSystem</plugin>
+      </xacro:if>
+      <xacro:unless value="$(arg use_fake_hardware)">
+        <param name="robot_ip">${robot_ip}</param>
+        <plugin>hardware_interface/VelocityJointInterface</plugin>
+        <param name="gear_ratio">24</param>
+        <param name="canbus_dev">can0</param>
+        <param name="encoder_cpr">10</param>
+        <param name="flip_motor_direction">0</param> <!-- 1/0 instead of true/false -->
+        <param name="gains_p">0.025</param>
+        <param name="gains_i">0.005</param>
+        <param name="gains_d">0.0</param>
+      </xacro:unless>
+    </hardware>
+    <joint name="left_wheel">
+      <command_interface name="velocity">
+        <param name="min">-3.15</param>
+        <param name="max">3.15</param>
+      </command_interface>
+      <state_interface name="position"/>
+      <state_interface name="velocity"/>
+    </joint>
+    <joint name="right_wheel">
+      <command_interface name="velocity">
+        <param name="min">-3.15</param>
+        <param name="max">3.15</param>
+      </command_interface>
+      <state_interface name="position"/>
+      <state_interface name="velocity"/>
+    </joint>
+  </ros2_control>
   <!-- Bring in simulation data for Gazebo. -->
   <xacro:include filename="$(find ridgeback_description)/urdf/ridgeback.gazebo" />

Commit message: current state of onboard pc

File: ridgeback_description/urdf/accessories.urdf.xacro (robot description, xacro)
@@ -4,11 +4,11 @@
     As you add to this URDF, please be aware that both the robot and
     simulation include it. You must retain compatibility with all of
-    the following launch files:
+    the following launch files
     ridgeback_viz/launch/view_model.launch
     ridgeback_gazebo/launch/ridgeback_world.launch
     ridgeback_base/launch/base.launch
   -->
-  <xacro:include filename="$(find ridgeback_description)/urdf/accessories/sick_lms1xx_mount.urdf.xacro" />
-  <xacro:include filename="$(find ridgeback_description)/urdf/accessories/sick_s300_mount.urdf.xacro" />
+<!--  <xacro:include filename="$(find ridgeback_description)/urdf/accessories/sick_lms1xx_mount.urdf.xacro" />-->
+  <!-- xacro:include filename="$(find ridgeback_description)/urdf/accessories/sick_s300_mount.urdf.xacro" / -->
   <xacro:include filename="$(find ridgeback_description)/urdf/accessories/hokuyo_ust-10lx_mount.urdf.xacro" />
   <!-- If enabled, generate the front HOKUYO UST-10LX LASER payload. -->
@@ -25,23 +25,23 @@
   </xacro:if>
   <!-- If enabled, generate the front SICK LMS111 LASER payload. -->
-  <xacro:if value="$(optenv RIDGEBACK_FRONT_SICK_LASER 0)">
+<!--  <xacro:if value="$(optenv RIDGEBACK_FRONT_SICK_LASER 0)">
     <xacro:sick_lms1xx_mount prefix="front"
                              topic="front/scan"
                              location="1" />
-  </xacro:if>
+  </xacro:if>-->
   <!-- If enabled, generate the rear SICK LMS111 LASER payload. -->
-  <xacro:if value="$(optenv RIDGEBACK_REAR_SICK_LASER 0)">
+<!--  <xacro:if value="$(optenv RIDGEBACK_REAR_SICK_LASER 0)">
     <xacro:sick_lms1xx_mount prefix="rear"
                              topic="rear/scan"
                              location="-1" />
-  </xacro:if>
+  </xacro:if>-->
   <!-- If enabled, generate the front SICK S300 LASER payload.
        This uses the same mesh as the lms1xx since they are the footprint
        and the simulation parameters can be variable. -->
-  <xacro:if value="$(optenv RIDGEBACK_FRONT_S300_LASER 0)">
+  <!-- xacro:if value="$(optenv RIDGEBACK_FRONT_S300_LASER 0)">
     <xacro:sick_s300_mount prefix="front"
                              topic="front/scan"
                              location="1" />
-  </xacro:if>
+  </xacro:if -->
   <!-- If enabled, generate the rear SICK S300 LASER payload. -->
   <xacro:if value="$(optenv RIDGEBACK_REAR_S300_LASER 0)">

File: ridgeback_description/urdf/ridgeback.urdf.xacro (robot description, xacro)
@@ -1,4 +1,5 @@
 <?xml version="1.0"?>
 <robot name="ridgeback" xmlns:xacro="http://ros.org/wiki/xacro">
+  <xacro:arg name="use_fake_hardware" default="true"/>
   <xacro:property name="PI" value="3.1415926535897931" />
   <xacro:property name="wheel_radius" value="0.0759" />
@@ -21,4 +22,13 @@
   <material name="yellow"><color rgba="0.8 0.8 0.0 1.0" /></material>
   <material name="black"><color rgba="0.15 0.15 0.15 1.0" /></material>
+  <!-- ros2 control include -->
+  <!-- xacro:include filename="$(find ridgeback_description)/urdf/ridgeback.ros2_control.xacro" /-->
+  <!-- ros2 control instance -->
+  <!-- xacro:ridgeback_ros2_control
+    name="ridgeback_ros2_control" prefix="${prefix}"
+    side="${side}"
+    use_fake_hardware="$(arg use_fake_hardware)"
+    initial_positions="${initial_positions}"
+    robot_ip="$(arg robot_ip)" /-->
   <xacro:macro name="wheel" params="prefix side *joint_pose">
     <link name="${prefix}_${side}_wheel_link">
@@ -51,5 +61,5 @@
       <axis xyz="0 1 0" />
     </joint>
-    <transmission name="${prefix}_wheel_trans">
+<!--    <transmission name="${prefix}_wheel_trans">
       <type>transmission_interface/SimpleTransmission</type>
       <joint name="${prefix}_${side}_wheel">
@@ -59,5 +69,5 @@
         <mechanicalReduction>1</mechanicalReduction>
       </actuator>
-    </transmission>
+    </transmission>-->
   </xacro:macro>
   <xacro:macro name="rocker" params="prefix joint_type location *joint_limits">
@@ -264,4 +274,54 @@
     <origin xyz="0 0 ${deck_height}" rpy="0 0 0"/>
   </joint>
+  <ros2_control name="ridgeback_hardware" type="system">
+    <hardware>
+      <xacro:if value="$(arg use_fake_hardware)">
+        <plugin>fake_components/GenericSystem</plugin>
+      </xacro:if>
+      <xacro:unless value="$(arg use_fake_hardware)">
+        <param name="robot_ip">${robot_ip}</param>
+        <plugin>ridgeback_base/RidgebackHardware</plugin>
+        <param name="gear_ratio">24</param>
+        <param name="canbus_dev">can0</param>
+        <param name="encoder_cpr">10</param>
+        <param name="flip_motor_direction">0</param> <!-- 1/0 instead of true/false -->
+        <param name="gains_p">0.025</param>
+        <param name="gains_i">0.005</param>
+        <param name="gains_d">0.0</param>
+      </xacro:unless>
+    </hardware>
+    <joint name="front_left_wheel">
+      <command_interface name="velocity">
+        <param name="min">-3.15</param>
+        <param name="max">3.15</param>
+      </command_interface>
+      <state_interface name="position"/>
+      <state_interface name="velocity"/>
+    </joint>
+    <joint name="front_right_wheel">
+      <command_interface name="velocity">
+        <param name="min">-3.15</param>
+        <param name="max">3.15</param>
+      </command_interface>
+      <state_interface name="position"/>
+      <state_interface name="velocity"/>
+    </joint>
+    <joint name="rear_left_wheel">
+      <command_interface name="velocity">
+        <param name="min">-3.15</param>
+        <param name="max">3.15</param>
+      </command_interface>
+      <state_interface name="position"/>
+      <state_interface name="velocity"/>
+    </joint>
+    <joint name="rear_right_wheel">
+      <command_interface name="velocity">
+        <param name="min">-3.15</param>
+        <param name="max">3.15</param>
+      </command_interface>
+      <state_interface name="position"/>
+      <state_interface name="velocity"/>
+    </joint>
+  </ros2_control>
   <!-- Bring in simulation data for Gazebo. -->
   <xacro:include filename="$(find ridgeback_description)/urdf/ridgeback.gazebo" />
@@ -271,4 +331,4 @@
   <xacro:include filename="$(find ridgeback_description)/urdf/accessories.urdf.xacro" />
   <!-- Optional custom includes. -->
-  <xacro:include filename="$(optenv RIDGEBACK_URDF_EXTRAS empty.urdf)" />
+<!--  <xacro:include filename="$(optenv RIDGEBACK_URDF_EXTRAS empty.urdf)" />-->
 </robot>
