Commit message: the diff drive comes up nicely, currently commented out to continue tshooting mecanum driver. considering borrowing a found mecanum driver controller

File: ridgeback_description/urdf/ridgeback.urdf.xacro (robot description, xacro)
@@ -291,5 +291,5 @@
       </xacro:unless>
     </hardware>
-    <joint name="left_wheel">
+    <joint name="front_left_wheel">
       <command_interface name="velocity">
         <param name="min">-3.15</param>
@@ -299,5 +299,21 @@
       <state_interface name="velocity"/>
     </joint>
-    <joint name="right_wheel">
+    <joint name="front_right_wheel">
+      <command_interface name="velocity">
+        <param name="min">-3.15</param>
+        <param name="max">3.15</param>
+      </command_interface>
+      <state_interface name="position"/>
+      <state_interface name="velocity"/>
+    </joint>
+    <joint name="rear_left_wheel">
+      <command_interface name="velocity">
+        <param name="min">-3.15</param>
+        <param name="max">3.15</param>
+      </command_interface>
+      <state_interface name="position"/>
+      <state_interface name="velocity"/>
+    </joint>
+    <joint name="rear_right_wheel">
       <command_interface name="velocity">
         <param name="min">-3.15</param>

Commit message: gazebo loads but commands are not followed, plugin work to commence

File: ridgeback_description/urdf/ridgeback.urdf.xacro (robot description, xacro)
@@ -1,5 +1,6 @@
 <?xml version="1.0"?>
 <robot name="ridgeback" xmlns:xacro="http://ros.org/wiki/xacro">
-  <xacro:arg name="use_fake_hardware" default="true"/>
+  <xacro:arg name="physical_robot" default="false"/>
+  <xacro:arg name="control_yaml_file" default=""/>
   <xacro:property name="PI" value="3.1415926535897931" />
   <xacro:property name="wheel_radius" value="0.0759" />
@@ -61,13 +62,9 @@
       <axis xyz="0 1 0" />
     </joint>
-<!--    <transmission name="${prefix}_wheel_trans">
-      <type>transmission_interface/SimpleTransmission</type>
-      <joint name="${prefix}_${side}_wheel">
-        <hardwareInterface>hardware_interface/VelocityJointInterface</hardwareInterface>
-      </joint>
-      <actuator name="${prefix}_${side}_actuator">
-        <mechanicalReduction>1</mechanicalReduction>
-      </actuator>
-    </transmission>-->
+    <gazebo reference="${prefix}_${side}_wheel_link">
+      <material>Gazebo/DarkGrey</material>
+      <mu1 value="0.0"/>
+      <mu2 value="0.0"/>
+    </gazebo>
   </xacro:macro>
   <xacro:macro name="rocker" params="prefix joint_type location *joint_limits">
@@ -276,8 +273,8 @@
   <ros2_control name="ridgeback_hardware" type="system">
     <hardware>
-      <xacro:if value="$(arg use_fake_hardware)">
+      <xacro:unless value="$(arg physical_robot)">
         <plugin>fake_components/GenericSystem</plugin>
-      </xacro:if>
-      <xacro:unless value="$(arg use_fake_hardware)">
+      </xacro:unless>
+      <xacro:if value="$(arg physical_robot)">
         <param name="robot_ip">${robot_ip}</param>
         <plugin>ridgeback_base/RidgebackHardware</plugin>
@@ -289,5 +286,5 @@
         <param name="gains_i">0.005</param>
         <param name="gains_d">0.0</param>
-      </xacro:unless>
+      </xacro:if>
     </hardware>
     <joint name="front_left_wheel">
@@ -325,9 +322,12 @@
   </ros2_control>
   <!-- Bring in simulation data for Gazebo. -->
-  <xacro:include filename="$(find ridgeback_description)/urdf/ridgeback.gazebo" />
+<!--  <xacro:include filename="$(find ridgeback_description)/urdf/ridgeback.gazebo" />-->
+  <xacro:unless value="$(arg physical_robot)">
+    <xacro:include filename="$(find ridgeback_description)/urdf/ridgeback-temp.gazebo" />
+  </xacro:unless>
   <!-- Optional standard accessories, including their simulation data. The rendering
        of these into the final description is controlled by optenv variables, which
        default each one to off.-->
-  <xacro:include filename="$(find ridgeback_description)/urdf/accessories.urdf.xacro" />
+<!--  <xacro:include filename="$(find ridgeback_description)/urdf/accessories.urdf.xacro" />-->
   <!-- Optional custom includes. -->
 <!--  <xacro:include filename="$(optenv RIDGEBACK_URDF_EXTRAS empty.urdf)" />-->

Commit message: ridgeback controllable in gazebo using diff drive controller

File: ridgeback_description/urdf/ridgeback.urdf.xacro (robot description, xacro)
@@ -32,4 +32,67 @@
     initial_positions="${initial_positions}"
     robot_ip="$(arg robot_ip)" /-->
+  <link name="base_link"></link>
+  <joint name="base_link_joint" type="fixed">
+    <origin xyz="0 0 0" rpy="0 0 0" />
+    <parent link="base_link"/>
+    <child link="chassis_link" />
+  </joint>
+  <link name="chassis_link">
+    <visual>
+      <origin xyz="0 0 0" rpy="0 0 0" />
+      <geometry>
+        <mesh filename="package://ridgeback_description/meshes/body.stl"/>
+      </geometry>
+      <material name="black" />
+    </visual>
+    <collision>
+      <origin xyz="0 0 0"/>
+      <geometry>
+        <mesh filename="package://ridgeback_description/meshes/body-collision.stl"/>
+      </geometry>
+    </collision>
+    <inertial>
+      <origin xyz="0.012 0.002 0.067" rpy="${PI/2} 0 ${PI/2}"/>
+      <mass value="165.304"/>
+      <inertia
+        ixx="4.4744" ixy="0.03098" ixz="0.003647"
+        iyy="7.1624" iyz="0.1228"
+        izz="4.6155"/>
+    </inertial>
+  </link>
+  <joint name="top_link_joint" type="fixed">
+    <origin xyz="0 0 0" rpy="0 0 0" />
+    <parent link="chassis_link"/>
+    <child link="top_link" />
+  </joint>
+  <link name="top_link">
+    <visual>
+      <origin xyz="0 0 0" rpy="0 0 0" />
+      <geometry>
+        <mesh filename="package://ridgeback_description/meshes/top.stl" />
+      </geometry>
+      <material name="black" />
+    </visual>
+    <collision>
+      <origin xyz="0 0 0" rpy="0 0 0" />
+      <geometry>
+        <mesh filename="package://ridgeback_description/meshes/top.stl"/>
+      </geometry>
+    </collision>
+  </link>
+  <joint name="axle_joint" type="fixed">
+    <origin xyz="0 0 ${axle_offset}" rpy="0 0 0" />
+    <parent link="chassis_link"/>
+    <child link="axle_link" />
+  </joint>
+  <link name="axle_link">
+    <visual>
+      <origin xyz="0 0 0" rpy="0 ${PI/2} 0" />
+      <geometry>
+        <mesh filename="package://ridgeback_description/meshes/axle.stl" />
+      </geometry>
+      <material name="black" />
+    </visual>
+  </link>
   <xacro:macro name="wheel" params="prefix side *joint_pose">
     <link name="${prefix}_${side}_wheel_link">
@@ -63,7 +126,11 @@
     </joint>
     <gazebo reference="${prefix}_${side}_wheel_link">
-      <material>Gazebo/DarkGrey</material>
-      <mu1 value="0.0"/>
-      <mu2 value="0.0"/>
+    <material>Gazebo/DarkGrey</material>
+    <selfCollide>false</selfCollide>
+    <mu1 value="0.5"/> <!-- mu1 & mu2 are normally 0 for this platform -->
+    <mu2 value="0.5"/>
+    <kp value="10000000.0" />
+    <kd value="1" />
+    <fdir1 value="1 0 0"/>
     </gazebo>
   </xacro:macro>
@@ -100,39 +167,13 @@
     </xacro:wheel>
   </xacro:macro>
-  <xacro:rocker prefix="front" joint_type="revolute" location="1" >
+  <xacro:rocker prefix="front" joint_type="fixed" location="1" >
+    <limit effort="0" velocity="0" />
+  </xacro:rocker>
+<!--  <xacro:rocker prefix="front" joint_type="revolute" location="1" >
     <limit lower="-0.08726" upper="0.08726" effort="0" velocity="0" />
-  </xacro:rocker>
+  </xacro:rocker> This isn't working currently, wondering if it's a typo-->
   <xacro:rocker prefix="rear" joint_type="fixed" location="-1" >
     <limit effort="0" velocity="0" />
   </xacro:rocker>
-  <link name="base_link"></link>
-  <joint name="base_link_joint" type="fixed">
-    <origin xyz="0 0 0" rpy="0 0 0" />
-    <parent link="base_link"/>
-    <child link="chassis_link" />
-  </joint>
-  <link name="chassis_link">
-    <visual>
-      <origin xyz="0 0 0" rpy="0 0 0" />
-      <geometry>
-        <mesh filename="package://ridgeback_description/meshes/body.stl"/>
-      </geometry>
-      <material name="black" />
-    </visual>
-    <collision>
-      <origin xyz="0 0 0"/>
-      <geometry>
-        <mesh filename="package://ridgeback_description/meshes/body-collision.stl"/>
-      </geometry>
-    </collision>
-    <inertial>
-      <origin xyz="0.012 0.002 0.067" rpy="${PI/2} 0 ${PI/2}"/>
-      <mass value="165.304"/>
-      <inertia
-        ixx="4.4744" ixy="0.03098" ixz="0.003647"
-        iyy="7.1624" iyz="0.1228"
-        izz="4.6155"/>
-    </inertial>
-  </link>
   <joint name="right_side_cover_link_joint" type="fixed">
     <origin xyz="0 0 0" rpy="0 0 0" />
@@ -217,38 +258,4 @@
       </geometry>
       <material name="red" />
-    </visual>
-  </link>
-  <joint name="top_link_joint" type="fixed">
-    <origin xyz="0 0 0" rpy="0 0 0" />
-    <parent link="chassis_link"/>
-    <child link="top_link" />
-  </joint>
-  <link name="top_link">
-    <visual>
-      <origin xyz="0 0 0" rpy="0 0 0" />
-      <geometry>
-        <mesh filename="package://ridgeback_description/meshes/top.stl" />
-      </geometry>
-      <material name="black" />
-    </visual>
-    <collision>
-      <origin xyz="0 0 0" rpy="0 0 0" />
-      <geometry>
-        <mesh filename="package://ridgeback_description/meshes/top.stl"/>
-      </geometry>
-    </collision>
-  </link>
-  <joint name="axle_joint" type="fixed">
-    <origin xyz="0 0 ${axle_offset}" rpy="0 0 0" />
-    <parent link="chassis_link"/>
-    <child link="axle_link" />
-  </joint>
-  <link name="axle_link">
-    <visual>
-      <origin xyz="0 0 0" rpy="0 ${PI/2} 0" />
-      <geometry>
-        <mesh filename="package://ridgeback_description/meshes/axle.stl" />
-      </geometry>
-      <material name="black" />
     </visual>
   </link>
@@ -274,5 +281,5 @@
     <hardware>
       <xacro:unless value="$(arg physical_robot)">
-        <plugin>fake_components/GenericSystem</plugin>
+        <plugin>gazebo_ros2_control/GazeboSystem</plugin> <!-- instead of fake_components/GenericSystem -->
       </xacro:unless>
       <xacro:if value="$(arg physical_robot)">
